Commit message: Add gps_common package and reindent xml xacro files

File: pablo_uav_system_ws/src/thirdparty/summit_xl/robotnik_sensors/urdf/gps.urdf.xacro (robot description, xacro)
@@ -1,54 +1,56 @@
 <?xml version="1.0"?>
 <robot name="sensor_gps" xmlns:xacro="http://ros.org/wiki/xacro">
-  <xacro:macro name="sensor_gps" params="name parent *origin">
-	  <!-- ANTENNA GPS -->
-	  <joint name="${name}_joint" type="fixed">
-	    <axis xyz="0 1 0"/>
-	    <xacro:insert_block name="origin"/>
-	    <parent link="${parent}"/>
-	    <child link="${name}_link"/>
-	  </joint>
-	  <link name="${name}_link">
-	    <inertial>
-	      <mass value="0.001"/>
-	      <origin rpy="0 0 0" xyz="0 0 0"/>
-	      <inertia ixx="0.0001" ixy="0" ixz="0" iyy="0.000001" iyz="0" izz="0.0001"/>
-	    </inertial>
-	    <visual>
-	      <origin rpy="0 0 0" xyz="0 0 0"/>
-	      <material name="gps_color">
-           <color rgba="1 1 1 1"/>
-        </material>
-	      <geometry>
-	        <mesh filename="package://robotnik_sensors/meshes/antenna_3GO16.stl" scale="1.0 1.0 1.0"/>
-	      </geometry>
-	    </visual>
-	    <collision>
-	      <origin rpy="0 0 0" xyz="0 0 0"/>
-	      <geometry>
-	        <mesh filename="package://robotnik_sensors/meshes/antenna_3GO16.stl" scale="1.0 1.0 1.0"/>
-	      </geometry>
-	    </collision>
-	  </link>
-	  <gazebo reference="${name}_link">
-	    <material>Gazebo/White</material>
-	    <gravity>true</gravity>
-	  </gazebo>
-    <gazebo>
-      <plugin name="${name}_link" filename="libhector_gazebo_ros_gps.so">
-        <alwaysOn>1</alwaysOn>
-				<updateRate>10.0</updateRate>
-				<bodyName>base_footprint</bodyName>
-				<topicName>mavros/gps/fix</topicName>
-				<!-- Robotnik position-->
-				<referenceLatitude>39.493800</referenceLatitude>
-				<referenceLongitude>-0.377982</referenceLongitude>
-				<velocityTopicName>fix_velocity</velocityTopicName>
-				<drift>5.0 5.0 5.0</drift>
-				<gaussianNoise>0.1 0.1 0.1</gaussianNoise>
-				<velocityDrift>0 0 0</velocityDrift>
-				<velocityGaussianNoise>0.1 0.1 0.1</velocityGaussianNoise>
-      </plugin>
-		</gazebo>
-  </xacro:macro>
+    <xacro:macro name="sensor_gps" params="name parent *origin">
+        <!-- ANTENNA GPS -->
+        <joint name="${name}_joint" type="fixed">
+            <axis xyz="0 1 0"/>
+            <xacro:insert_block name="origin"/>
+            <parent link="${parent}"/>
+            <child link="${name}_link"/>
+        </joint>
+        <link name="${name}_link">
+            <inertial>
+                <mass value="0.001"/>
+                <origin rpy="0 0 0" xyz="0 0 0"/>
+                <inertia ixx="0.0001" ixy="0" ixz="0" iyy="0.000001" iyz="0" izz="0.0001"/>
+            </inertial>
+            <visual>
+                <origin rpy="0 0 0" xyz="0 0 0"/>
+                <material name="gps_color">
+                    <color rgba="1 1 1 1"/>
+                </material>
+                <geometry>
+                    <mesh filename="package://robotnik_sensors/meshes/antenna_3GO16.stl" scale="1.0 1.0 1.0"/>
+                </geometry>
+            </visual>
+            <collision>
+                <origin rpy="0 0 0" xyz="0 0 0"/>
+                <geometry>
+                    <mesh filename="package://robotnik_sensors/meshes/antenna_3GO16.stl" scale="1.0 1.0 1.0"/>
+                </geometry>
+            </collision>
+        </link>
+        <gazebo reference="${name}_link">
+            <material>Gazebo/White</material>
+            <gravity>true</gravity>
+        </gazebo>
+        <gazebo>
+            <plugin name="${name}_link" filename="libhector_gazebo_ros_gps.so">
+                <alwaysOn>1</alwaysOn>
+                <updateRate>10.0</updateRate>
+                <bodyName>base_footprint</bodyName>
+                <topicName>mavros/gps/fix</topicName>
+                <!-- Robotnik position-->
+                <!--<referenceLatitude>39.493800</referenceLatitude>-->
+                <!--<referenceLongitude>-0.377982</referenceLongitude>-->
+                <referenceLatitude>0</referenceLatitude>
+                <referenceLongitude>0</referenceLongitude>
+                <velocityTopicName>fix_velocity</velocityTopicName>
+                <drift>5.0 5.0 5.0</drift>
+                <gaussianNoise>0.1 0.1 0.1</gaussianNoise>
+                <velocityDrift>0 0 0</velocityDrift>
+                <velocityGaussianNoise>0.1 0.1 0.1</velocityGaussianNoise>
+            </plugin>
+        </gazebo>
+    </xacro:macro>
 </robot>

File: pablo_uav_system_ws/src/thirdparty/summit_xl/summit_xl_common/summit_xl_description/robots/summit_xl.urdf.xacro (robot description, xacro)
@@ -1,106 +1,90 @@
 <?xml version="1.0"?>
 <robot name="summit_xl" xmlns:xacro="http://www.ros.org/wiki/xacro">
-	<!-- ***************** -->
-	<!-- Imported elements -->
-	<!-- ***************** -->
-	<!-- First we import all posible elements defined in the urdf.xacro files. All these elements are defined as macro:xacros -->
-	<!-- Import summit XL base elements -->
-	<xacro:include filename="$(find summit_xl_description)/urdf/bases/summit_xl_base.urdf.xacro" />
-	<!-- Import summit XL wheels -->
-	<xacro:include filename="$(find summit_xl_description)/urdf/wheels/rubber_wheel.urdf.xacro" />
-	<!-- Import all available sensors -->
-	<!--
-	<xacro:include filename="$(find robotnik_sensors)/urdf/all_sensors.urdf.xacro" />
-	-->
-  	<!-- Import the landing platform on which quadrotors can easily land -->
-  	<xacro:include filename="$(find summit_xl_description)/urdf/platform/platform_cylinder.urdf.xacro" />
+    <!-- ***************** -->
+    <!-- Imported elements -->
+    <!-- ***************** -->
+    <!-- First we import all posible elements defined in the urdf.xacro files. All these elements are defined as macro:xacros -->
+    <!-- Import summit XL base elements -->
+    <xacro:include filename="$(find summit_xl_description)/urdf/bases/summit_xl_base.urdf.xacro" />
+    <!-- Import summit XL wheels -->
+    <xacro:include filename="$(find summit_xl_description)/urdf/wheels/rubber_wheel.urdf.xacro" />
+    <!--Import all available sensors-->
+    <xacro:include filename="$(find robotnik_sensors)/urdf/all_sensors.urdf.xacro" />
+    <!-- Import the landing platform on which quadrotors can easily land -->
+    <xacro:include filename="$(find summit_xl_description)/urdf/platform/platform_cylinder.urdf.xacro" />
     <xacro:include filename="$(find summit_xl_description)/urdf/platform/landing_platform.urdf.xacro" />
     <xacro:include filename="$(find summit_xl_description)/urdf/platform/landing_indicator.urdf.xacro" />
-	<!-- ***************** -->
-	<!-- Global parameters -->
-	<!-- ***************** -->
-	<xacro:property name="PI" value="3.1415926535897931"/>
-	<!-- Wheel parameters -->
-	<xacro:property name="wheel_offset_x" value="0.229" />    <!-- x,y,z in translation from base_link to the center of the wheel -->
-	<xacro:property name="wheel_offset_y" value="0.234" />
-	<xacro:property name="wheel_offset_z" value="0.0" />
-	<!-- Flag to select the high or low quality model -->
-	<xacro:property name="hq" value="true" />
-	<!-- *************** -->
-	<!-- Robots Elements -->
-	<!-- *************** -->
-	<!-- Here we create the robot elements using the xacro:macros imported at the beggining of this file -->
-	<!-- Summit XL base -->
-	<xacro:summit_xl_base name="summit_xl" publish_bf="true" hq="${hq}" />
-	<!-- Gazebo ros control pluggins -->
-	<xacro:ros_control/>
-	<!-- Gazebo skid steering pluggins -->
-	<xacro:skid_steering broadcastOdomTF="1"/>
-	<!-- WHEELS -->
-	<xacro:rubber_wheel name="front_right" parent="base_link" reflect="false" hq="${hq}">
-		<origin xyz="${wheel_offset_x} -${wheel_offset_y} ${wheel_offset_z}" rpy="0 0 0"/>
-	</xacro:rubber_wheel>
-	<xacro:rubber_wheel name="front_left" parent="base_link" reflect="true" hq="${hq}">
-		<origin xyz="${wheel_offset_x} ${wheel_offset_y} ${wheel_offset_z}" rpy="0 0 0"/>
-	</xacro:rubber_wheel>
-	<xacro:rubber_wheel name="back_left" parent="base_link" reflect="true" hq="${hq}">
-		<origin xyz="-${wheel_offset_x} ${wheel_offset_y} ${wheel_offset_z}" rpy="0 0 0"/>
-	</xacro:rubber_wheel>
-	<xacro:rubber_wheel name="back_right" parent="base_link" reflect="false" hq="${hq}">
-		<origin xyz="-${wheel_offset_x} -${wheel_offset_y} ${wheel_offset_z}" rpy="0 0 0"/>
-	</xacro:rubber_wheel>
-	<!-- LANDING PLATFORM-->
-	<xacro:platform_cylinder name="platform_cylinder" parent="base_link" >
-		<origin xyz="0.0 0.0 0.325" rpy="0 0 0"/>
-	</xacro:platform_cylinder>
-	<xacro:landing_platform name="landing_platform" parent="platform_cylinder" >
-		<origin xyz="0.0 0.0 0.05" rpy="0 0 0"/>
-	</xacro:landing_platform>
-	<xacro:landing_indicator name="landing_indicator" parent="landing_platform" >
-		<origin xyz="0.6 0.0 0.0" rpy="0 0 0"/>
-	</xacro:landing_indicator>
-	<!-- SENSORS -->
-  <!-- Hokuyo laser sensors can be parametized with min_angle and max_angle e.g: -->
-  <!--xacro:sensor_hokuyo_utm30lx name="hokuyo_base" parent="base_link" min_angle="2.35" max_angle="-2.35"-->
-<!--
-	<xacro:sensor_hokuyo_utm30lx name="hokuyo_base" parent="base_link">
-		<origin xyz="0.0 0.0 0.33" rpy="0 0 0"/>
-	</xacro:sensor_hokuyo_utm30lx>
--->
-<!--
-	<xacro:sensor_hokuyo_urg04lx name="hokuyo1" parent="base_link">
-		<origin xyz="-0.1 0.0 0.33" rpy="0 0 0"/>
-	</xacro:sensor_hokuyo_urg04lx>
--->
-<!--
-  <xacro:sensor_hokuyo_ust10lx name="hokuyo_base" parent="base_link">
-		<origin xyz="0.0 0.0 0.33" rpy="0 0 0"/>
-	</xacro:sensor_hokuyo_ust10lx>
--->
-    <!--
-	<xacro:sensor_axis name="camera" parent="base_link">
-		<origin xyz="0.19 0 0.17" rpy="0 ${15*PI/180} 0"/>
-	</xacro:sensor_axis>
-	<xacro:sensor_imu name="imu" parent="base_link">
-		<origin xyz="-0.18 0.0 0.170" rpy="0 0 0"/>
-	</xacro:sensor_imu>
-	<xacro:sensor_gps name="gps" parent="base_link">
-		<origin xyz="-0.22 0 0.275" rpy="0 0 0"/>
-	</xacro:sensor_gps>
--->
-<!--
-	<xacro:sensor_asus_xtion_pro name="xtion_pro" parent="base_link">
-		<origin xyz="0.3 0.0 0.3" rpy="0 0 0"/>
-	</xacro:sensor_asus_xtion_pro>
--->
-<!--
-	<xacro:sensor_kinect name="kinect" parent="base_link">
-		<origin xyz="0.325 0.0 0.16" rpy="0 0 0"/>
-	</xacro:sensor_kinect>
--->
-<!--
-	<xacro:sensor_fotonic name="fotonic" parent="base_link">
-		<origin xyz="0.3 0.0 0.24" rpy="0 0 0"/>
-	</xacro:sensor_fotonic>
--->
+    <!-- ***************** -->
+    <!-- Global parameters -->
+    <!-- ***************** -->
+    <xacro:property name="PI" value="3.1415926535897931"/>
+    <!-- Wheel parameters -->
+    <xacro:property name="wheel_offset_x" value="0.229" />    <!-- x,y,z in translation from base_link to the center of the wheel -->
+    <xacro:property name="wheel_offset_y" value="0.234" />
+    <xacro:property name="wheel_offset_z" value="0.0" />
+    <!-- Flag to select the high or low quality model -->
+    <xacro:property name="hq" value="true" />
+    <!-- *************** -->
+    <!-- Robots Elements -->
+    <!-- *************** -->
+    <!-- Here we create the robot elements using the xacro:macros imported at the beggining of this file -->
+    <!-- Summit XL base -->
+    <xacro:summit_xl_base name="summit_xl" publish_bf="true" hq="${hq}" />
+    <!-- Gazebo ros control pluggins -->
+    <xacro:ros_control/>
+    <!-- Gazebo skid steering pluggins -->
+    <xacro:skid_steering broadcastOdomTF="1"/>
+    <!-- WHEELS -->
+    <xacro:rubber_wheel name="front_right" parent="base_link" reflect="false" hq="${hq}">
+        <origin xyz="${wheel_offset_x} -${wheel_offset_y} ${wheel_offset_z}" rpy="0 0 0"/>
+    </xacro:rubber_wheel>
+    <xacro:rubber_wheel name="front_left" parent="base_link" reflect="true" hq="${hq}">
+        <origin xyz="${wheel_offset_x} ${wheel_offset_y} ${wheel_offset_z}" rpy="0 0 0"/>
+    </xacro:rubber_wheel>
+    <xacro:rubber_wheel name="back_left" parent="base_link" reflect="true" hq="${hq}">
+        <origin xyz="-${wheel_offset_x} ${wheel_offset_y} ${wheel_offset_z}" rpy="0 0 0"/>
+    </xacro:rubber_wheel>
+    <xacro:rubber_wheel name="back_right" parent="base_link" reflect="false" hq="${hq}">
+        <origin xyz="-${wheel_offset_x} -${wheel_offset_y} ${wheel_offset_z}" rpy="0 0 0"/>
+    </xacro:rubber_wheel>
+    <!-- LANDING PLATFORM-->
+    <xacro:platform_cylinder name="platform_cylinder" parent="base_link" >
+        <origin xyz="0.0 0.0 0.325" rpy="0 0 0"/>
+    </xacro:platform_cylinder>
+    <xacro:landing_platform name="landing_platform" parent="platform_cylinder" >
+        <origin xyz="0.0 0.0 0.05" rpy="0 0 0"/>
+    </xacro:landing_platform>
+    <xacro:landing_indicator name="landing_indicator" parent="landing_platform" >
+        <origin xyz="0.6 0.0 0.0" rpy="0 0 0"/>
+    </xacro:landing_indicator>
+    <!-- SENSORS -->
+    <!-- Hokuyo laser sensors can be parametized with min_angle and max_angle e.g: -->
+    <!--xacro:sensor_hokuyo_utm30lx name="hokuyo_base" parent="base_link" min_angle="2.35" max_angle="-2.35"-->
+    <!--<xacro:sensor_hokuyo_utm30lx name="hokuyo_base" parent="base_link">-->
+        <!--<origin xyz="0.0 0.0 0.33" rpy="0 0 0"/>-->
+    <!--</xacro:sensor_hokuyo_utm30lx>-->
+    <!--<xacro:sensor_hokuyo_urg04lx name="hokuyo1" parent="base_link">-->
+        <!--<origin xyz="-0.1 0.0 0.33" rpy="0 0 0"/>-->
+    <!--</xacro:sensor_hokuyo_urg04lx>-->
+    <!--<xacro:sensor_hokuyo_ust10lx name="hokuyo_base" parent="base_link">-->
+        <!--<origin xyz="0.0 0.0 0.33" rpy="0 0 0"/>-->
+    <!--</xacro:sensor_hokuyo_ust10lx>-->
+    <!--<xacro:sensor_axis name="camera" parent="base_link">-->
+        <!--<origin xyz="0.19 0 0.17" rpy="0 ${15*PI/180} 0"/>-->
+    <!--</xacro:sensor_axis>-->
+    <!--<xacro:sensor_imu name="imu" parent="base_link">-->
+        <!--<origin xyz="-0.18 0.0 0.170" rpy="0 0 0"/>-->
+    <!--</xacro:sensor_imu>-->
+    <xacro:sensor_gps name="gps" parent="base_link">
+        <origin xyz="-0.22 0 0.275" rpy="0 0 0"/>
+    </xacro:sensor_gps>
+    <!--<xacro:sensor_asus_xtion_pro name="xtion_pro" parent="base_link">-->
+        <!--<origin xyz="0.3 0.0 0.3" rpy="0 0 0"/>-->
+    <!--</xacro:sensor_asus_xtion_pro>-->
+    <!--<xacro:sensor_kinect name="kinect" parent="base_link">-->
+        <!--<origin xyz="0.325 0.0 0.16" rpy="0 0 0"/>-->
+    <!--</xacro:sensor_kinect>-->
+    <!--<xacro:sensor_fotonic name="fotonic" parent="base_link">-->
+        <!--<origin xyz="0.3 0.0 0.24" rpy="0 0 0"/>-->
+    <!--</xacro:sensor_fotonic>-->
 </robot>

File: pablo_uav_system_ws/src/thirdparty/tum_simulator/cvg_sim_gazebo_plugins/urdf/quadrotor_sensors.urdf.xacro (robot description, xacro)
@@ -1,67 +1,67 @@
 <?xml version="1.0"?>
 <robot xmlns:sensor="http://playerstage.sourceforge.net/gazebo/xmlschema/#sensor"
-xmlns:controller="http://playerstage.sourceforge.net/gazebo/xmlschema/#controller"
-xmlns:interface="http://playerstage.sourceforge.net/gazebo/xmlschema/#interface"
-xmlns:xacro="http://ros.org/wiki/xacro"
->
+    xmlns:controller="http://playerstage.sourceforge.net/gazebo/xmlschema/#controller"
+    xmlns:interface="http://playerstage.sourceforge.net/gazebo/xmlschema/#interface"
+    xmlns:xacro="http://ros.org/wiki/xacro"
+    >
   <!-- Quadrotor Sensor Plugins
-        <frameId>ardrone_base_link</frameId>
--->
-  <xacro:macro name="quadrotor_sensors">
-    <gazebo>
-      <plugin name="quadrotor_imu_sim" filename="libhector_gazebo_ros_imu.so">
-        <alwaysOn>true</alwaysOn>
-        <updateRate>100.0</updateRate>
-        <bodyName>base_link</bodyName>
-        <frameId>ardrone_base_link</frameId>
-        <topicName>/ardrone/imu</topicName>
-        <rpyOffsets>0 0 0</rpyOffsets> <!-- deprecated -->
-        <gaussianNoise>0</gaussianNoise>  <!-- deprecated -->
-        <accelDrift>0.5 0.5 0.5</accelDrift>
-        <accelGaussianNoise>0.35 0.35 0.3</accelGaussianNoise>
-        <rateDrift>0.0 0.0 0.0</rateDrift>
-        <rateGaussianNoise>0.00 0.00 0.00</rateGaussianNoise>
-        <headingDrift>0.0</headingDrift>
-        <headingGaussianNoise>0.00</headingGaussianNoise>
-      </plugin>
-      <plugin name="quadrotor_baro_sim" filename="libhector_gazebo_ros_baro.so">
-        <alwaysOn>true</alwaysOn>
-        <updateRate>10.0</updateRate>
-        <bodyName>base_link</bodyName>
-        <topicName>/ardrone/pressure_height</topicName>
-        <altimeterTopicName>/ardrone/altimeter</altimeterTopicName>
-        <offset>0</offset>
-        <drift>0.0</drift>
-        <gaussianNoise>0.0</gaussianNoise>
-      </plugin>
-      <plugin name="quadrotor_magnetic_sim" filename="libhector_gazebo_ros_magnetic.so">
-        <alwaysOn>true</alwaysOn>
-        <updateRate>10.0</updateRate>
-        <bodyName>base_link</bodyName>
-        <topicName>/ardrone/magnetic</topicName>
-        <offset>0 0 0</offset>
-        <drift>0.0 0.0 0.0</drift>
-        <gaussianNoise>1.3e-2 1.3e-2 1.3e-2</gaussianNoise>
-      </plugin>
-      <plugin name="quadrotor_gps_sim" filename="libhector_gazebo_ros_gps.so">
-        <alwaysOn>true</alwaysOn>
-        <updateRate>4.0</updateRate>
-        <bodyName>base_link</bodyName>
-        <topicName>/ardrone/fix</topicName>
-        <velocityTopicName>/ardrone/fix_velocity</velocityTopicName>
-        <drift>5.0 5.0 5.0</drift>
-        <gaussianNoise>0.1 0.1 0.1</gaussianNoise>
-        <velocityDrift>0 0 0</velocityDrift>
-        <velocityGaussianNoise>0.1 0.1 0.1</velocityGaussianNoise>
-      </plugin>
-      <plugin name="quadrotor_groundtruth_sim" filename="libgazebo_ros_p3d.so">
-        <alwaysOn>true</alwaysOn>
-        <updateRate>100.0</updateRate>
-        <bodyName>base_link</bodyName>
-        <topicName>/ardrone/ground_truth/state</topicName>
-        <gaussianNoise>0.0</gaussianNoise>
-        <frameName>map</frameName>
-      </plugin>
-    </gazebo>
-  </xacro:macro>
-</robot>
+      <frameId>ardrone_base_link</frameId>
+  -->
+      <xacro:macro name="quadrotor_sensors">
+          <gazebo>
+              <plugin name="quadrotor_imu_sim" filename="libhector_gazebo_ros_imu.so">
+                  <alwaysOn>true</alwaysOn>
+                  <updateRate>100.0</updateRate>
+                  <bodyName>base_link</bodyName>
+                  <frameId>ardrone_base_link</frameId>
+                  <topicName>/ardrone/imu</topicName>
+                  <rpyOffsets>0 0 0</rpyOffsets> <!-- deprecated -->
+                  <gaussianNoise>0</gaussianNoise>  <!-- deprecated -->
+                  <accelDrift>0.5 0.5 0.5</accelDrift>
+                  <accelGaussianNoise>0.35 0.35 0.3</accelGaussianNoise>
+                  <rateDrift>0.0 0.0 0.0</rateDrift>
+                  <rateGaussianNoise>0.00 0.00 0.00</rateGaussianNoise>
+                  <headingDrift>0.0</headingDrift>
+                  <headingGaussianNoise>0.00</headingGaussianNoise>
+              </plugin>
+              <plugin name="quadrotor_baro_sim" filename="libhector_gazebo_ros_baro.so">
+                  <alwaysOn>true</alwaysOn>
+                  <updateRate>10.0</updateRate>
+                  <bodyName>base_link</bodyName>
+                  <topicName>/ardrone/pressure_height</topicName>
+                  <altimeterTopicName>/ardrone/altimeter</altimeterTopicName>
+                  <offset>0</offset>
+                  <drift>0.0</drift>
+                  <gaussianNoise>0.0</gaussianNoise>
+              </plugin>
+              <plugin name="quadrotor_magnetic_sim" filename="libhector_gazebo_ros_magnetic.so">
+                  <alwaysOn>true</alwaysOn>
+                  <updateRate>10.0</updateRate>
+                  <bodyName>base_link</bodyName>
+                  <topicName>/ardrone/magnetic</topicName>
+                  <offset>0 0 0</offset>
+                  <drift>0.0 0.0 0.0</drift>
+                  <gaussianNoise>1.3e-2 1.3e-2 1.3e-2</gaussianNoise>
+              </plugin>
+              <plugin name="quadrotor_gps_sim" filename="libhector_gazebo_ros_gps.so">
+                  <alwaysOn>true</alwaysOn>
+                  <updateRate>4.0</updateRate>
+                  <bodyName>base_link</bodyName>
+                  <topicName>/ardrone/fix</topicName>
+                  <velocityTopicName>/ardrone/fix_velocity</velocityTopicName>
+                  <drift>5.0 5.0 5.0</drift>
+                  <gaussianNoise>0.1 0.1 0.1</gaussianNoise>
+                  <velocityDrift>0 0 0</velocityDrift>
+                  <velocityGaussianNoise>0.1 0.1 0.1</velocityGaussianNoise>
+              </plugin>
+              <plugin name="quadrotor_groundtruth_sim" filename="libgazebo_ros_p3d.so">
+                  <alwaysOn>true</alwaysOn>
+                  <updateRate>100.0</updateRate>
+                  <bodyName>base_link</bodyName>
+                  <topicName>/ardrone/ground_truth/state</topicName>
+                  <gaussianNoise>0.0</gaussianNoise>
+                  <frameName>map</frameName>
+              </plugin>
+          </gazebo>
+      </xacro:macro>
+  </robot>
