Commit message: Add GPS sensor to helipad rover in the file summit_xl.urdf.xacro

File: catkin_ws/src/summit_xl/robotnik_sensors/urdf/gps.urdf.xacro (robot description, xacro)
@@ -1,54 +1,54 @@
 <?xml version="1.0"?>
 <robot name="sensor_gps" xmlns:xacro="http://ros.org/wiki/xacro">
-  <xacro:macro name="sensor_gps" params="name parent *origin">
-	  <!-- ANTENNA GPS -->
-	  <joint name="${name}_joint" type="fixed">
-	    <axis xyz="0 1 0"/>
-	    <xacro:insert_block name="origin"/>
-	    <parent link="${parent}"/>
-	    <child link="${name}_link"/>
-	  </joint>
-	  <link name="${name}_link">
-	    <inertial>
-	      <mass value="0.001"/>
-	      <origin rpy="0 0 0" xyz="0 0 0"/>
-	      <inertia ixx="0.0001" ixy="0" ixz="0" iyy="0.000001" iyz="0" izz="0.0001"/>
-	    </inertial>
-	    <visual>
-	      <origin rpy="0 0 0" xyz="0 0 0"/>
-	      <material name="gps_color">
-           <color rgba="1 1 1 1"/>
-        </material>
-	      <geometry>
-	        <mesh filename="package://robotnik_sensors/meshes/antenna_3GO16.stl" scale="1.0 1.0 1.0"/>
-	      </geometry>
-	    </visual>
-	    <collision>
-	      <origin rpy="0 0 0" xyz="0 0 0"/>
-	      <geometry>
-	        <mesh filename="package://robotnik_sensors/meshes/antenna_3GO16.stl" scale="1.0 1.0 1.0"/>
-	      </geometry>
-	    </collision>
-	  </link>
-	  <gazebo reference="${name}_link">
-	    <material>Gazebo/White</material>
-	    <gravity>true</gravity>
-	  </gazebo>
-    <gazebo>
-      <plugin name="${name}_link" filename="libhector_gazebo_ros_gps.so">
-        <alwaysOn>1</alwaysOn>
-				<updateRate>10.0</updateRate>
-				<bodyName>base_footprint</bodyName>
-				<topicName>mavros/gps/fix</topicName>
-				<!-- Robotnik position-->
-				<referenceLatitude>39.493800</referenceLatitude>
-				<referenceLongitude>-0.377982</referenceLongitude>
-				<velocityTopicName>fix_velocity</velocityTopicName>
-				<drift>5.0 5.0 5.0</drift>
-				<gaussianNoise>0.1 0.1 0.1</gaussianNoise>
-				<velocityDrift>0 0 0</velocityDrift>
-				<velocityGaussianNoise>0.1 0.1 0.1</velocityGaussianNoise>
-      </plugin>
-		</gazebo>
-  </xacro:macro>
+    <xacro:macro name="sensor_gps" params="name parent *origin">
+        <!-- ANTENNA GPS -->
+        <joint name="${name}_joint" type="fixed">
+            <axis xyz="0 1 0"/>
+            <xacro:insert_block name="origin"/>
+            <parent link="${parent}"/>
+            <child link="${name}_link"/>
+        </joint>
+        <link name="${name}_link">
+            <inertial>
+                <mass value="0.001"/>
+                <origin rpy="0 0 0" xyz="0 0 0"/>
+                <inertia ixx="0.0001" ixy="0" ixz="0" iyy="0.000001" iyz="0" izz="0.0001"/>
+            </inertial>
+            <visual>
+                <origin rpy="0 0 0" xyz="0 0 0"/>
+                <material name="gps_color">
+                    <color rgba="1 1 1 1"/>
+                </material>
+                <geometry>
+                    <mesh filename="package://robotnik_sensors/meshes/antenna_3GO16.stl" scale="1.0 1.0 1.0"/>
+                </geometry>
+            </visual>
+            <collision>
+                <origin rpy="0 0 0" xyz="0 0 0"/>
+                <geometry>
+                    <mesh filename="package://robotnik_sensors/meshes/antenna_3GO16.stl" scale="1.0 1.0 1.0"/>
+                </geometry>
+            </collision>
+        </link>
+        <gazebo reference="${name}_link">
+            <material>Gazebo/White</material>
+            <gravity>true</gravity>
+        </gazebo>
+        <gazebo>
+            <plugin name="${name}_link" filename="libhector_gazebo_ros_gps.so">
+                <alwaysOn>1</alwaysOn>
+                <updateRate>10.0</updateRate>
+                <bodyName>base_footprint</bodyName>
+                <topicName>mavros/gps/fix</topicName>
+                <!-- Robotnik position-->
+                <referenceLatitude>39.493800</referenceLatitude>
+                <referenceLongitude>-0.377982</referenceLongitude>
+                <velocityTopicName>fix_velocity</velocityTopicName>
+                <drift>5.0 5.0 5.0</drift>
+                <gaussianNoise>0.1 0.1 0.1</gaussianNoise>
+                <velocityDrift>0 0 0</velocityDrift>
+                <velocityGaussianNoise>0.1 0.1 0.1</velocityGaussianNoise>
+            </plugin>
+        </gazebo>
+    </xacro:macro>
 </robot>
