Commit message: fix tum simulator for kinetic and comment at set TIME_WITHOUT_SEEING to max

File: pablo_uav_system_ws/src/thirdparty/tum_simulator/cvg_sim_gazebo/urdf/quadrotor.urdf.xacro (robot description, xacro)
@@ -3,5 +3,6 @@
     xmlns:sensor="http://playerstage.sourceforge.net/gazebo/xmlschema/#sensor"
     xmlns:controller="http://playerstage.sourceforge.net/gazebo/xmlschema/#controller"
-    xmlns:xacro="http://ros.org/wiki/xacro">
+    xmlns:interface="http://playerstage.sourceforge.net/gazebo/xmlschema/#interface"
+    xmlns:xacro="http://playerstage.sourceforge.net/gazebo/xmlschema/#interface">
     <!-- Included URDF Files -->
     <xacro:include filename="$(find cvg_sim_gazebo)/urdf/quadrotor_base.urdf.xacro" />

File: pablo_uav_system_ws/src/thirdparty/tum_simulator/cvg_sim_gazebo/urdf/quadrotor_base.urdf.xacro (robot description, xacro)
@@ -2,14 +2,12 @@
 <robot xmlns:sensor="http://playerstage.sourceforge.net/gazebo/xmlschema/#sensor"
 xmlns:controller="http://playerstage.sourceforge.net/gazebo/xmlschema/#controller"
-xmlns:xacro="http://ros.org/wiki/xacro">
+xmlns:interface="http://playerstage.sourceforge.net/gazebo/xmlschema/#interface"
+xmlns:xacro="http://ros.org/wiki/xacro"
+>
   <xacro:include filename="$(find cvg_sim_gazebo_plugins)/urdf/quadrotor_plugins.urdf.xacro" />
+  <property name="pi" value="3.1415926535897931" />
   <!-- Main quadrotor link -->
   <xacro:macro name="quadrotor_base_macro">
     <link name="base_link">
-      <inertial>
-        <mass value="1.477" />
-        <origin xyz="0 0 0" />
-        <inertia ixx="0.01152" ixy="0.0" ixz="0.0" iyy="0.01152" iyz="0.0" izz="0.0218" />
-      </inertial>
       <visual>
         <origin xyz="0 0 0" rpy="0 0 0" />
@@ -25,7 +23,17 @@
       </collision>
     </link>
+    <link name="dummy_link">
+	      <inertial>
+        	<mass value="1.477" />
+        	<origin xyz="0 0 0" />
+        	<inertia ixx="0.01152" ixy="0.0" ixz="0.0" iyy="0.01152" iyz="0.0" izz="0.0218" />
+      	      </inertial>
+    </link>
+    <joint name="dummy_joint" type="fixed">
+ 	 <parent link="base_link"/>
+         <child link="dummy_link"/>
+    </joint>
     <gazebo reference="base_link">
       <turnGravityOff>false</turnGravityOff>
-      <!-- <gravity>false</gravity> -->
     </gazebo>
     <!-- Gazebo Plugins -->

File: pablo_uav_system_ws/src/thirdparty/tum_simulator/cvg_sim_gazebo/urdf/quadrotor_sensors.urdf.xacro (robot description, xacro)
@@ -3,6 +3,7 @@
 xmlns:sensor="http://playerstage.sourceforge.net/gazebo/xmlschema/#sensor"
 xmlns:controller="http://playerstage.sourceforge.net/gazebo/xmlschema/#controller"
-xmlns:xacro="http://ros.org/wiki/xacro">
-    <xacro:property name="M_PI" value="3.1415926535897931" />
+xmlns:interface="http://playerstage.sourceforge.net/gazebo/xmlschema/#interface"
+xmlns:xacro="http://playerstage.sourceforge.net/gazebo/xmlschema/#interface">
+    <property name="M_PI" value="3.1415926535897931" />
     <!-- Included URDF Files -->
     <xacro:include filename="$(find cvg_sim_gazebo)/urdf/quadrotor_base.urdf.xacro" />
@@ -27,6 +28,6 @@
     <!-- Downward facing camera -->
     <xacro:include filename="$(find cvg_sim_gazebo)/urdf/sensors/generic_camera.urdf.xacro" />
-    <xacro:generic_camera name="bottom" sim_name="ardrone" parent="base_link" update_rate="60" res_x="640" res_y="480" image_format="R8G8B8" hfov="${100*M_PI/180}">
-        <origin xyz="0.15 0.0 0.0" rpy="0 ${M_PI/2} 0"/>
+    <xacro:generic_camera name="bottom" sim_name="ardrone" parent="base_link" update_rate="60" res_x="640" res_y="360" image_format="R8G8B8" hfov="${81*M_PI/180}">
+      <origin xyz="0.15 0.0 0.0" rpy="0 ${M_PI/2} 0"/>
     </xacro:generic_camera>
 </robot>

File: pablo_uav_system_ws/src/thirdparty/tum_simulator/cvg_sim_gazebo/urdf/sensors/generic_camera.urdf.xacro (robot description, xacro)
@@ -2,9 +2,11 @@
 <robot xmlns:sensor="http://playerstage.sourceforge.net/gazebo/xmlschema/#sensor"
 xmlns:controller="http://playerstage.sourceforge.net/gazebo/xmlschema/#controller"
-xmlns:xacro="http://ros.org/wiki/xacro">
-    <xacro:property name="M_PI" value="3.1415926535897931" />
+xmlns:interface="http://playerstage.sourceforge.net/gazebo/xmlschema/#interface"
+  xmlns:xacro="http://ros.org/wiki/xacro"
+  >
+    <property name="M_PI" value="3.1415926535897931" />
     <xacro:macro name="generic_camera" params="name sim_name parent *origin update_rate res_x res_y image_format hfov">
       <joint name="${name}_joint" type="fixed">
-        <xacro:insert_block name="origin" />
+        <insert_block name="origin" />
         <parent link="${parent}"/>
         <child link="${name}_link"/>
@@ -82,6 +84,5 @@
         </plugin>
       </sensor>
-      <turnGravityOff>true</turnGravityOff>
-      <material>PR2/Blue</material>
+      <material>Gazebo/Blue</material>
     </gazebo>
     </xacro:macro>

File: pablo_uav_system_ws/src/thirdparty/tum_simulator/cvg_sim_gazebo/urdf/sensors/hokuyo_utm30lx.urdf.xacro (robot description, xacro)
@@ -2,8 +2,10 @@
 <robot xmlns:sensor="http://playerstage.sourceforge.net/gazebo/xmlschema/#sensor"
 xmlns:controller="http://playerstage.sourceforge.net/gazebo/xmlschema/#controller"
-xmlns:xacro="http://ros.org/wiki/xacro">
+xmlns:interface="http://playerstage.sourceforge.net/gazebo/xmlschema/#interface"
+  xmlns:xacro="http://ros.org/wiki/xacro"
+  >
     <xacro:macro name="hokuyo_utm30lx" params="name parent *origin ros_topic update_rate ray_count min_angle max_angle">
       <joint name="${name}_joint" type="fixed">
-	<xacro:insert_block name="origin" />
+	<insert_block name="origin" />
 	<parent link="${parent}"/>
 	<child link="${name}_frame"/>

File: pablo_uav_system_ws/src/thirdparty/tum_simulator/cvg_sim_gazebo/urdf/sensors/sonar_sensor.urdf.xacro (robot description, xacro)
@@ -2,5 +2,7 @@
 <robot xmlns:sensor="http://playerstage.sourceforge.net/gazebo/xmlschema/#sensor"
 xmlns:controller="http://playerstage.sourceforge.net/gazebo/xmlschema/#controller"
-xmlns:xacro="http://ros.org/wiki/xacro">
+xmlns:interface="http://playerstage.sourceforge.net/gazebo/xmlschema/#interface"
+xmlns:xacro="http://ros.org/wiki/xacro"
+>
   <xacro:macro name="sonar_sensor" params="name parent *origin ros_topic update_rate min_range max_range field_of_view ray_count">
     <joint name="${name}_joint" type="fixed">
@@ -53,4 +55,7 @@
         <plugin name="gazebo_ros_${name}_controller" filename="libhector_gazebo_ros_sonar.so">
           <gaussianNoise>0.000</gaussianNoise>
+          <offset>0.0 </offset>
+          <drift>0.0</drift>
+	  <driftFrequency>0.0</driftFrequency>
           <topicName>${ros_topic}</topicName>
           <frameId>${name}_link</frameId>

File: pablo_uav_system_ws/src/thirdparty/tum_simulator/cvg_sim_gazebo_plugins/urdf/quadrotor_sensors.urdf.xacro (robot description, xacro)
@@ -1,67 +1,79 @@
 <?xml version="1.0"?>
 <robot xmlns:sensor="http://playerstage.sourceforge.net/gazebo/xmlschema/#sensor"
-    xmlns:controller="http://playerstage.sourceforge.net/gazebo/xmlschema/#controller"
-    xmlns:interface="http://playerstage.sourceforge.net/gazebo/xmlschema/#interface"
-    xmlns:xacro="http://ros.org/wiki/xacro"
-    >
+xmlns:controller="http://playerstage.sourceforge.net/gazebo/xmlschema/#controller"
+xmlns:interface="http://playerstage.sourceforge.net/gazebo/xmlschema/#interface"
+xmlns:xacro="http://ros.org/wiki/xacro"
+>
   <!-- Quadrotor Sensor Plugins
-      <frameId>ardrone_base_link</frameId>
-  -->
-      <xacro:macro name="quadrotor_sensors">
-          <gazebo>
-              <plugin name="quadrotor_imu_sim" filename="libhector_gazebo_ros_imu.so">
-                  <alwaysOn>true</alwaysOn>
-                  <updateRate>100.0</updateRate>
-                  <bodyName>base_link</bodyName>
-                  <frameId>ardrone_base_link</frameId>
-                  <topicName>/ardrone/imu</topicName>
-                  <rpyOffsets>0 0 0</rpyOffsets> <!-- deprecated -->
-                  <gaussianNoise>0</gaussianNoise>  <!-- deprecated -->
-                  <accelDrift>0.5 0.5 0.5</accelDrift>
-                  <accelGaussianNoise>0.35 0.35 0.3</accelGaussianNoise>
-                  <rateDrift>0.0 0.0 0.0</rateDrift>
-                  <rateGaussianNoise>0.00 0.00 0.00</rateGaussianNoise>
-                  <headingDrift>0.0</headingDrift>
-                  <headingGaussianNoise>0.00</headingGaussianNoise>
-              </plugin>
-              <plugin name="quadrotor_baro_sim" filename="libhector_gazebo_ros_baro.so">
-                  <alwaysOn>true</alwaysOn>
-                  <updateRate>10.0</updateRate>
-                  <bodyName>base_link</bodyName>
-                  <topicName>/ardrone/pressure_height</topicName>
-                  <altimeterTopicName>/ardrone/altimeter</altimeterTopicName>
-                  <offset>0</offset>
-                  <drift>0.0</drift>
-                  <gaussianNoise>0.0</gaussianNoise>
-              </plugin>
-              <plugin name="quadrotor_magnetic_sim" filename="libhector_gazebo_ros_magnetic.so">
-                  <alwaysOn>true</alwaysOn>
-                  <updateRate>10.0</updateRate>
-                  <bodyName>base_link</bodyName>
-                  <topicName>/ardrone/magnetic</topicName>
-                  <offset>0 0 0</offset>
-                  <drift>0.0 0.0 0.0</drift>
-                  <gaussianNoise>1.3e-2 1.3e-2 1.3e-2</gaussianNoise>
-              </plugin>
-              <plugin name="quadrotor_gps_sim" filename="libhector_gazebo_ros_gps.so">
-                  <alwaysOn>true</alwaysOn>
-                  <updateRate>4.0</updateRate>
-                  <bodyName>base_link</bodyName>
-                  <topicName>/ardrone/fix</topicName>
-                  <velocityTopicName>/ardrone/fix_velocity</velocityTopicName>
-                  <drift>5.0 5.0 5.0</drift>
-                  <gaussianNoise>0.1 0.1 0.1</gaussianNoise>
-                  <velocityDrift>0 0 0</velocityDrift>
-                  <velocityGaussianNoise>0.1 0.1 0.1</velocityGaussianNoise>
-              </plugin>
-              <plugin name="quadrotor_groundtruth_sim" filename="libgazebo_ros_p3d.so">
-                  <alwaysOn>true</alwaysOn>
-                  <updateRate>100.0</updateRate>
-                  <bodyName>base_link</bodyName>
-                  <topicName>/ardrone/ground_truth/state</topicName>
-                  <gaussianNoise>0.0</gaussianNoise>
-                  <frameName>map</frameName>
-              </plugin>
-          </gazebo>
-      </xacro:macro>
-  </robot>
+        <frameId>ardrone_base_link</frameId>
+-->
+  <xacro:macro name="quadrotor_sensors">
+    <gazebo>
+      <plugin name="quadrotor_imu_sim" filename="libhector_gazebo_ros_imu.so">
+        <alwaysOn>true</alwaysOn>
+        <updateRate>100.0</updateRate>
+        <bodyName>base_link</bodyName>
+        <frameId>ardrone_base_link</frameId>
+        <topicName>/ardrone/imu</topicName>
+        <rpyOffsets>0 0 0</rpyOffsets> <!-- deprecated -->
+        <gaussianNoise>0</gaussianNoise>  <!-- deprecated -->
+        <accelDrift>0.5 0.5 0.5</accelDrift>
+        <accelGaussianNoise>0.35 0.35 0.3</accelGaussianNoise>
+        <rateDrift>0.0 0.0 0.0</rateDrift>
+        <rateGaussianNoise>0.00 0.00 0.00</rateGaussianNoise>
+        <headingDrift>0.0</headingDrift>
+	<headingDriftFrequency>0.0</headingDriftFrequency>
+	<headingOffset>0.0	</headingOffset>
+	<rateDriftFrequency>0 0 0</rateDriftFrequency>
+	<rateOffset>0 0 0</rateOffset>
+	<accelDriftFrequency>0 0 0</accelDriftFrequency>
+	<accelOffset>0 0 0</accelOffset>
+        <headingGaussianNoise>0.00</headingGaussianNoise>
+      </plugin>
+      <plugin name="quadrotor_baro_sim" filename="libhector_gazebo_ros_baro.so">
+        <alwaysOn>true</alwaysOn>
+        <updateRate>10.0</updateRate>
+        <bodyName>base_link</bodyName>
+        <topicName>/ardrone/pressure_height</topicName>
+        <altimeterTopicName>/ardrone/altimeter</altimeterTopicName>
+        <offset>0</offset>
+        <drift>0.1</drift>
+	<driftFrequency>0.0</driftFrequency>
+        <gaussianNoise>0.5</gaussianNoise>
+      </plugin>
+      <plugin name="quadrotor_magnetic_sim" filename="libhector_gazebo_ros_magnetic.so">
+        <alwaysOn>true</alwaysOn>
+        <updateRate>10.0</updateRate>
+        <bodyName>base_link</bodyName>
+        <topicName>/ardrone/magnetic</topicName>
+        <offset>0 0 0</offset>
+        <drift>0.0 0.0 0.0</drift>
+	<driftFrequency>0.0 0.0 0.0</driftFrequency>
+        <gaussianNoise>1.3e-2 1.3e-2 1.3e-2</gaussianNoise>
+      </plugin>
+      <plugin name="quadrotor_gps_sim" filename="libhector_gazebo_ros_gps.so">
+        <alwaysOn>true</alwaysOn>
+        <updateRate>4.0</updateRate>
+        <bodyName>base_link</bodyName>
+        <topicName>/ardrone/fix</topicName>
+        <velocityTopicName>/ardrone/fix_velocity</velocityTopicName>
+	<offset>0 0 0</offset>
+        <drift>5.0 5.0 5.0</drift>
+	<driftFrequency>0.0 0.0 0.0</driftFrequency>
+        <gaussianNoise>0.1 0.1 0.1</gaussianNoise>
+        <velocityDrift>0 0 0</velocityDrift>
+        <velocityDriftFrequency>0 0 0</velocityDriftFrequency>
+        <velocityGaussianNoise>0.1 0.1 0.1</velocityGaussianNoise>
+	<velocityOffset>0 0 0</velocityOffset>
+      </plugin>
+      <plugin name="quadrotor_groundtruth_sim" filename="libgazebo_ros_p3d.so">
+        <alwaysOn>true</alwaysOn>
+        <updateRate>100.0</updateRate>
+        <bodyName>base_link</bodyName>
+        <topicName>/ardrone/ground_truth/state</topicName>
+        <gaussianNoise>0.0</gaussianNoise>
+        <frameName>map</frameName>
+      </plugin>
+    </gazebo>
+  </xacro:macro>
+</robot>

File: pablo_uav_system_ws/src/thirdparty/tum_simulator/cvg_sim_gazebo_plugins/urdf/quadrotor_simple_controller.urdf.xacro (robot description, xacro)
@@ -25,9 +25,9 @@
         <velocityZProportionalGain>5.0</velocityZProportionalGain>
         <velocityZDifferentialGain>1.0</velocityZDifferentialGain>
-        <velocityZLimit>5.0</velocityZLimit> <!-- 0.5 -->
+        <velocityZLimit>5.0</velocityZLimit>
         <maxForce>30</maxForce>
-        <motionSmallNoise>0.0</motionSmallNoise> <!-- 0.05 -->
-        <motionDriftNoise>0.0</motionDriftNoise> <!-- 0.03 -->
-        <motionDriftNoiseTime>0.0</motionDriftNoiseTime> <!-- 5.0 -->
+        <motionSmallNoise>0.0</motionSmallNoise>
+        <motionDriftNoise>0.0</motionDriftNoise>
+        <motionDriftNoiseTime>0.0</motionDriftNoiseTime>
       </plugin>
       <!-- <plugin name="quadrotor_state_controller" filename="libhector_gazebo_quadrotor_state_controller.so">
